File: RiserBoard_PCB/RiserBoard.sch (KiCad schematic (older format))
At the start: 10 parts, among them J1 BUS1, J2 AudioJack3, J3 BUS2

Commit message: Made Naming of Pins consistent
Connections:
- net B_L renamed B_T
- net T_L renamed T_T
Changed lines of the file:
@@
 T_R
 Text Label 2700 4300 0    50   ~ 0
-T_L
+T_T
 Text Label 3500 4100 0    50   ~ 0
 T_S
@@
 T_R
 Text Label 3500 4300 0    50   ~ 0
-T_L
+T_T
 Text Label 7500 4300 2    50   ~ 0
-B_L
+B_T
 Text Label 7500 4100 2    50   ~ 0
 B_S
@@
 	7200 4300 7500 4300
 Text Label 6650 4300 2    50   ~ 0
-B_L
+B_T
 Text Label 6650 4200 2    50   ~ 0
 B_R
